File: hardware/kicad/coffee-scale/coffee-scale_version_2.kicad_sch (KiCad schematic)
At the start: 25 parts, among them J2 JS2, Q1 DMG3415U, U1 ESP32-S3, U2 HX711, U4 AP2112/RT9080-3.3, U5 MCP73831-2-MC, X1G$1 JSTPH, X1MT1 JSTPH, X1MT2 JSTPH

Commit message: Update schematic
Parts:
- removed C4: 4.7uF, symbol Device:C
- removed J2: JS2, symbol Connector:Conn_01x02_Pin
- removed JP2: SolderJumper_2_Bridged, symbol Jumper:SolderJumper_2_Bridged
- removed R5: R, symbol Device:R
- removed R6: 2k, symbol Device:R
- removed U3: ~, symbol Custom:UC8151D
- removed U5: MCP73831-2-MC, Package_DFN_QFN:DFN-8-1EP_3x2mm_P0.5mm_EP1.7x1.4mm, symbol Battery_Management:MCP73831-2-MC
- removed X1G$1: JSTPH, symbol Connector:Conn_01x02_Socket
- added J1: Conn_01x08, symbol Connector_Generic:Conn_01x08
- added J3: Conn_01x02, symbol Connector_Generic:Conn_01x02
- added R3: 5.1k, symbol Device:R
- added U3: MCP73832-5-OT, Package_TO_SOT_SMD:SOT-23-5, symbol Battery_Management:MCP73832-5-OT
- C3: value 4.7uF -> 10uF
- R4: value 1k -> 5.1k
Connections:
- net 3.3V: now also J1.1 (Pin_1)
- net GND: now also R4.2, J1.8 (Pin_8), J3.1 (Pin_1), U3.2 (V_{SS})
- net VBAT: now also C3.1, J3.2 (Pin_2), U3.3 (V_{BAT})
- net VBUS: now also D2.2 (A), U3.4 (V_{DD}); no longer R4.2
- net at U1.39 (GPIO34): now also J1.2 (Pin_2)
- net at U1.40 (GPIO35): now also J1.3 (Pin_3)
- net at U1.41 (GPIO36): now also J1.4 (Pin_4)
- net at U1.42 (GPIO37): now also J1.5 (Pin_5)
- net at U1.43 (GPIO38): now also J1.6 (Pin_6)
- net at R4.1: now also U3.5 (PROG); no longer D2.2 (A)
- net +BATT: no longer names the net of D2.1 (K)
- net +BATT: now also R3.1; no longer C3.1
- new net: R3.2, U3.1 (STAT)
- no-connect marks 0 -> 54
Other:
- note added: "3V3"
- note added: "CLK"
- note added: "CS"
- note added: "D/C"
- note added: "DATA"
- note added: "RST"
- moved on the sheet: U1
