File: hardware/kicad/coffee-scale/coffee-scale.kicad_pcb (KiCad board)
At the start: 2 copper layers, 54 x 43.5 mm, 46 parts, among them J2 Conn_01x04, J3 Conn_01x02, J4 USB C, Q1 DMG3415U, Q2 S8550, SW1 SW_Push, SW2 SW_Push, SW3 SW_Push, U1 ESP32-S3, U2 HX711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

Commit message: .
Parts:
- Switch 1: renamed from SW1
- Switch 2: renamed from SW2
- Switch 3: renamed from SW3
- moved J3 1.25 mm to (136.0, 96.8)
- moved X1MT1 1.20 mm to (131.5, 95.8)
- moved X1MT2 1.20 mm to (124.5, 95.8)
- moved LS1 0.79 mm to (166.2, 102.8)
Routing:
- net 3.3V: track 86.8 -> 89.1 mm
- net Net-(D1-K): track 37.1 -> 39.1 mm
- net Net-(J3-Pin_2): track 6.83 -> 8.37 mm
- net /BUT3: track 32.4 -> 31.1 mm
- net Net-(U2-VFB): track 11.7 -> 13.1 mm
- net Net-(JP3-A): track 17.8 -> 16.8 mm
- net Net-(J1-Pin_6): track 41.2 -> 40.3 mm
- net GND: track 61.4 -> 60.6 mm
- net Net-(J1-Pin_5): track 36.5 -> 35.9 mm
Other:
- board size 54 x 43.5 mm -> 60 x 50 mm

Commit message: .
Parts:
- J1: renamed from OLED Display
- J3: footprint Connector_PinHeader_2.54mm:PinHeader_1x02_P2.54mm_Vertical -> Connector_JST:JST_PH_B2B-PH-K_1x02_P2.00mm_Vertical
- SW1: renamed from Switch 1
- SW2: renamed from Switch 2
- SW3: renamed from Switch 3
- U1: footprint Package_DFN_QFN:QFN-56-1EP_7x7mm_P0.4mm_EP4x4mm -> RF_Module:ESP32-S3-WROOM-1
- X1MT1: footprint Connector_JST:JST_PH_B2B-PH-K_1x02_P2.00mm_Vertical -> Connector_PinHeader_2.54mm:PinHeader_1x01_P2.54mm_Vertical
- moved X1MT2 74.8 mm to (188.9, 133.7), turned to 0 degrees
- moved U1 53.1 mm to (216.2, 109.8)
- moved J3 11.1 mm to (125.2, 94.0)
- moved X1MT1 5.51 mm to (128.2, 100.2)

Commit message: PCB Update
Parts:
- removed X1MT1: JSTPH, Connector_PinHeader_2.54mm:PinHeader_1x01_P2.54mm_Vertical
- removed X1MT2: JSTPH, Connector_JST:JST_PH_B2B-PH-K_1x02_P2.00mm_Vertical
- added C10: 20p, Capacitor_SMD:C_1206_3216Metric_Pad1.33x1.80mm_HandSolder, F.Cu at (170.5, 122.1)
- added C11: 20p, Capacitor_SMD:C_1206_3216Metric_Pad1.33x1.80mm_HandSolder, F.Cu at (173.9, 125.8)
- added D4: D_Schottky_Filled, Diode_SMD:D_SOD-123, F.Cu at (183.6, 100.8)
- added H1: MountingHole, MountingHole:MountingHole_2.5mm_Pad_TopBottom, F.Cu at (120.8, 96.8)
- added H2: MountingHole, MountingHole:MountingHole_2.5mm_Pad_TopBottom, F.Cu at (120.8, 132.0)
- added H3: MountingHole, MountingHole:MountingHole_2.5mm_Pad_TopBottom, F.Cu at (195.5, 96.5)
- added H4: MountingHole, MountingHole:MountingHole_2.5mm_Pad_TopBottom, F.Cu at (195.5, 132.0)
- added Q3: BSS138, Package_TO_SOT_SMD:SOT-23, F.Cu at (184.1, 103.8)
- added R11: 10k, Resistor_SMD:R_1206_3216Metric_Pad1.30x1.75mm_HandSolder, F.Cu at (180.0, 102.0)
- added R12: 22, Resistor_SMD:R_1206_3216Metric_Pad1.30x1.75mm_HandSolder, F.Cu at (173.0, 122.0)
- added R13: 22, Resistor_SMD:R_1206_3216Metric_Pad1.30x1.75mm_HandSolder, F.Cu at (175.2, 122.0)
- added TP6: TestPoint_Small, TestPoint:TestPoint_Pad_1.0x1.0mm, F.Cu at (125.2, 94.0)
- J3: footprint Connector_JST:JST_PH_B2B-PH-K_1x02_P2.00mm_Vertical -> Connector_JST:JST_PH_S2B-PH-K_1x02_P2.00mm_Horizontal
- J4: footprint Connector_USB:USB_C_Receptacle_GCT_USB4105-xx-A_16P_TopMnt_Horizontal -> Connector_USB:USB_C_Receptacle_GCT_USB4085
- R5, R6, R7, R8: value R -> 100
- moved U1 48.4 mm to (168.0, 106.0)
- moved LS1 27.3 mm to (192.8, 109.3)
- moved R5 23.0 mm to (148.9, 122.9)
- moved R6 23.0 mm to (148.9, 125.1)
- moved C8 23.0 mm to (147.5, 118.6)
- moved C9 23.0 mm to (150.0, 118.6)
- moved J2 23.0 mm to (144.5, 117.5)
- moved C7 22.8 mm to (152.8, 124.1)
- moved C4 22.5 mm to (157.0, 118.6), turned to 90 degrees
- moved TP1 22.3 mm to (190.8, 119.0)
- moved TP2 22.3 mm to (188.2, 119.0)
- moved TP3 22.3 mm to (185.8, 119.0)
- moved TP4 22.3 mm to (183.2, 119.0)
- moved TP5 22.3 mm to (180.8, 119.0)
- moved SW1 20.5 mm to (145.5, 131.0)
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Connections:
- J1 pad 1: 3.3V -> /CS
- J1 pad 2: Net-(J1-Pin_2) -> /RST
- J1 pad 3: Net-(J1-Pin_3) -> /D/C
- J1 pad 4: Net-(J1-Pin_4) -> /CLK
- J1 pad 5: Net-(J1-Pin_5) -> /DATA
- J1 pad 6: Net-(J1-Pin_6) -> 3.3V
- JP2 pad 2: /DATA -> Net-(JP2-B)
- LS1 pad 1: /BEEP -> 3.3V
- LS1 pad 2: GND -> Net-(D4-A)
- TP1 pad 1: Net-(J1-Pin_2) -> /CS
- TP2 pad 1: Net-(J1-Pin_3) -> /RST
- TP3 pad 1: Net-(J1-Pin_4) -> /D/C
- TP4 pad 1: Net-(J1-Pin_5) -> /CLK
- TP5 pad 1: Net-(J1-Pin_6) -> /DATA
- U1 pad 10: /DATA -> Net-(JP2-B)
- U1 pad 25: /D- -> Net-(U1-GPIO19/USB_D-)
- U1 pad 26: /D+ -> Net-(U1-GPIO20/USB_D+)
- U1 pad 39: Net-(J1-Pin_2) -> /CS
- U1 pad 40: Net-(J1-Pin_3) -> /RST
- U1 pad 41: Net-(J1-Pin_4) -> /D/C
Routing:
- net 3.3V: track 89.1 -> 0.00 mm, vias 2 -> 0
- net GND: track 60.6 -> 0.14 mm, vias 25 -> 0
- net VBUS: track 51.2 -> 0.00 mm, vias 4 -> 0
- net /BUT1: track 46.2 -> 0.00 mm, vias 2 -> 0
- net /BUT2: track 41.6 -> 0.00 mm, vias 4 -> 0
- net Net-(J1-Pin_6): track 40.3 -> 0.00 mm, vias 2 -> 0
- net Net-(D1-K): track 39.1 -> 0.00 mm, vias 2 -> 0
- net Net-(J1-Pin_5): track 35.9 -> 0.00 mm, vias 2 -> 0
- net Net-(J1-Pin_4): track 31.6 -> 0.00 mm, vias 2 -> 0
- net VBAT: track 31.5 -> 0.00 mm
- net /BUT3: track 31.1 -> 0.00 mm
- net Net-(J1-Pin_3): track 27.8 -> 0.00 mm, vias 2 -> 0
- net /D+: track 27.7 -> 0.00 mm, vias 2 -> 0
- net /E+: track 26.1 -> 0.00 mm, vias 2 -> 0
- net /D-: track 25.4 -> 0.00 mm, vias 2 -> 0
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- removed copper zone on B.Cu, net GND
Other:
- board size 60 x 50 mm -> 82.5 x 43 mm

Commit message: update
Parts:
- moved R2 20.7 mm to (141.5, 125.0), turned to -90 degrees
- moved J3 20.1 mm to (135.9, 118.5), turned to -90 degrees
- moved TP6 18.1 mm to (130.8, 111.2), turned to 90 degrees
- moved Q1 17.3 mm to (138.4, 124.9), turned to -90 degrees
- moved JP4 16.4 mm to (139.2, 119.0)
- moved U4 15.0 mm to (138.4, 129.1), turned to 90 degrees
- moved D2 13.4 mm to (139.2, 109.0), turned to 180 degrees
- moved H1 12.8 mm to (133.5, 96.2)
- moved H2 12.8 mm to (133.5, 132.0)
- moved R3 12.3 mm to (143.0, 105.8), turned to 90 degrees
- moved R9 10.4 mm to (139.3, 106.8), turned to 0 degrees
- moved C3 10.2 mm to (147.2, 108.4), turned to 0 degrees
- moved C2 10.2 mm to (135.5, 125.4), turned to 90 degrees
- moved R4 9.90 mm to (142.4, 100.8)
- moved R10 7.56 mm to (139.3, 104.5), turned to 0 degrees
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Routing:
- net 3.3V: track 0.00 -> 147.1 mm, vias 0 -> 9
- net Net-(Q2-B): track 0.00 -> 87.1 mm, vias 0 -> 4
- net /D+: track 0.00 -> 72.8 mm, vias 0 -> 1
- net /D-: track 0.00 -> 67.3 mm, vias 0 -> 8
- net VBUS: track 0.00 -> 55.1 mm
- net GND: track 0.14 -> 49.3 mm, vias 0 -> 29
- net /D/C: track 0.00 -> 44.6 mm, vias 0 -> 2
- net /E+: track 0.00 -> 43.9 mm, vias 0 -> 4
- net /CS: track 0.00 -> 41.3 mm, vias 0 -> 2
- net /RST: track 0.00 -> 38.9 mm, vias 0 -> 2
- net VBAT: track 0.00 -> 38.2 mm, vias 0 -> 3
- net Net-(D1-K): track 0.00 -> 36.7 mm
- net /BUT1: track 0.00 -> 27.4 mm
- net Net-(U2-VFB): track 2.00 -> 23.9 mm, vias 0 -> 2
- net Net-(U2-VBG): track 0.00 -> 19.5 mm, vias 0 -> 2
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- added copper zone on B.Cu, net GND
Other:
- board size 82.5 x 43 mm -> 70.2 x 43.2 mm

Commit message: logbook and PCB routing edits
Parts:
- moved H1 0.50 mm to (133.0, 96.2)
- moved H2 0.50 mm to (133.0, 132.0)
- moved J4 0.12 mm to (134.9, 101.8)
Routing:
- net Net-(Q2-B): track 87.1 -> 36.0 mm, vias 4 -> 3
- net Net-(U2-INA-): track 2.41 -> 40.8 mm
- net Net-(U2-INA+): track 4.01 -> 20.7 mm, vias 1 -> 2
- net /D+: track 72.8 -> 66.4 mm, vias 1 -> 5
- net Net-(U2-VBG): track 19.5 -> 13.8 mm, vias 2 -> 0
- net /RST: track 38.9 -> 44.6 mm
- net 3.3V: track 147.1 -> 152.6 mm, vias 9 -> 5
- net /CS: track 41.3 -> 45.5 mm, vias 2 -> 0
- net /D-: track 67.3 -> 71.2 mm, vias 8 -> 5
- net /BEEP: track 4.99 -> 8.52 mm
- net GND: track 49.3 -> 52.6 mm, vias 29 -> 30
- net /E+: track 43.9 -> 41.1 mm, vias 4 -> 2
- net Net-(D1-K): track 36.7 -> 39.1 mm
- net VBUS: track 55.1 -> 53.2 mm, vias 0 -> 2
- net /D/C: track 44.6 -> 43.1 mm
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
Commit message: Update coffee-scale.kicad_pcb
Parts:
- C1, C2, C5, C6: value 10μF -> 10uF
- D1: value MBR540 -> ~; footprint Diode_THT:D_DO-201AD_P15.24mm_Horizontal -> Diode_SMD:D_SOD-128
- D4: footprint Diode_SMD:D_SOD-123 -> Diode_SMD:D_SOD-128
- Q2: footprint Package_TO_SOT_THT:TO-92_Inline -> Package_TO_SOT_SMD:SOT-23-3
- SW1, SW2, SW3: footprint Button_Switch_SMD:SW_SPST_Omron_B3FS-105xP -> Button_Switch_SMD:SW_SPST_B3S-1000
- U4: footprint Package_TO_SOT_SMD:SOT-23-5 -> Package_TO_SOT_SMD:SOT-89-5_Handsoldering
- moved R6 8.59 mm to (145.0, 117.5), turned to 90 degrees
- moved R9 7.35 mm to (133.3, 111.0)
- moved C4 7.29 mm to (153.5, 112.2)
- moved C8 7.29 mm to (143.8, 112.3)
- moved C9 7.29 mm to (146.2, 112.3)
- moved R7 7.29 mm to (151.0, 112.2)
- moved R8 7.29 mm to (148.8, 112.3)
- moved C7 7.22 mm to (149.8, 117.5)
- moved C11 6.87 mm to (168.8, 121.2), turned to 0 degrees
- moved D4 6.81 mm to (184.5, 107.5), turned to -90 degrees
- moved J2 6.76 mm to (144.9, 124.5), turned to 90 degrees
- moved Q2 6.53 mm to (152.8, 116.9)
- moved D1 6.29 mm to (131.5, 113.8)
- moved R5 5.64 mm to (147.2, 117.5), turned to 90 degrees
- moved U4 2.32 mm to (137.8, 131.3)
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Routing:
- net Net-(U2-INA-): track 40.8 -> 16.1 mm, vias 0 -> 2
- net /D-: track 71.2 -> 52.7 mm, vias 5 -> 0
- net Net-(U2-VFB): track 24.1 -> 11.9 mm, vias 2 -> 0
- net 3.3V: track 152.6 -> 161.7 mm, vias 5 -> 6
- net /E+: track 41.1 -> 50.1 mm
- net Net-(J4-CC2): track 15.8 -> 6.77 mm
- net /S+: track 2.90 -> 11.9 mm, vias 0 -> 1
- net /D+: track 66.4 -> 57.5 mm, vias 5 -> 0
- net Net-(D1-K): track 39.1 -> 31.4 mm
- net Net-(D4-A): track 11.0 -> 18.0 mm
- net Net-(U4-EN): track 9.05 -> 15.5 mm
- net VBUS: track 53.2 -> 46.7 mm
- net Net-(J3-Pin_2): track 8.98 -> 3.27 mm, vias 2 -> 0
- net Net-(U2-VBG): track 13.8 -> 8.25 mm
- net Net-(Q3-G): track 10.3 -> 5.35 mm
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Other:
- board size 70.2 x 43.2 mm -> 71.5 x 43.2 mm
